File: Kicad/The Ear Tool.sch (KiCad schematic (older format))
At the start: 14 parts, among them P1 AUDIO-JACK-3F07-TRS, P2 Sensor Connector, P3 9V Battery Clip, SW1 Power Switch, SW2 Full Scope Switch, SW3 Gain Switch, U1 LM386

Commit message: Add files via upload
Parts:
- added C3: 0u1, Capacitor_SMD:C_0603_1608Metric, symbol Device:C_Small
- C1: footprint Capacitors_SMD:C_0805_HandSoldering -> Capacitor_SMD:C_0603_1608Metric
- C2: footprint Capacitors_THT:C_Radial_D5_L6_P2.5 -> Capacitor_SMD:CP_Elec_6.3x7.7
- D1: footprint Capacitors_SMD:C_0805 -> LED_THT:LED_D5.0mm_Clear
- LS1: footprint Oddities:NetTie-I_SMD -> SurfaceConnector:Surface Connector
- P1: footprint Connectors:AUDIO-JACK-3F07-TRS -> myFootprints:AUDIO-JACK-3F07-TRS; symbol The-Ear-Tool-rescue:AUDIO-JACK-3F07-TRS -> The-Ear-Tool-rescue:AUDIO-JACK-3F07-TRS-The-Ear-Tool-rescue
- P2: footprint Oddities:NetTie-I_SMD -> TerminalBlock_RND:TerminalBlock_RND_205-00232_Pitch5.08mm; symbol The-Ear-Tool-rescue:CONN_01X02 -> The-Ear-Tool-rescue:CONN_01X02-The-Ear-Tool-rescue
- P3: footprint Oddities:NetTie-I_SMD -> SurfaceConnector:Surface Connector; symbol The-Ear-Tool-rescue:CONN_01X02 -> The-Ear-Tool-rescue:CONN_01X02-The-Ear-Tool-rescue
- R1, R2: footprint Resistors_SMD:R_0805_HandSoldering -> Resistor_SMD:R_0603_1608Metric
- RV1: footprint myFootprints:POT_RV09_HORIZONTAL_WHO9 -> Potentiometer_THT:Potentiometer_Bourns_PTV09A-1_Single_Vertical; symbol The-Ear-Tool-rescue:POT -> The-Ear-Tool-rescue:POT-The-Ear-Tool-rescue
- SW1, SW2, SW3: footprint myFootprints:SW_SPDT_3P_11.1mm_5.5mm -> Switch:SPDT_generic_toggle; symbol Switch1:SW_DPDT_x2 -> The-Ear-Tool-rescue:SW_DPDT_x2-Switch1
- U1: symbol The-Ear-Tool-rescue:LM386 -> The-Ear-Tool-rescue:LM386-The-Ear-Tool-rescue
Other:
- moved on the sheet: D1, R1
Changed lines of the file:
@@
 EESchema Schematic File Version 4
-LIBS:The Ear Tool-cache
-EELAYER 29 0
+EELAYER 30 0
 EELAYER END
 $Descr A4 11693 8268
@@
 $EndDescr
 $Comp
-L The-Ear-Tool-rescue:LM386 U1
+L The-Ear-Tool-rescue:LM386-The-Ear-Tool-rescue U1
 U 1 1 5B89DD93
 P 5200 3400
@@
 F 0 "C2" V 6000 3350 50  0000 L CNN
 F 1 "220uF" V 5700 3250 50  0000 L CNN
-F 2 "Capacitors_THT:C_Radial_D5_L6_P2.5" H 5850 3400 50  0001 C CNN
+F 2 "Capacitor_SMD:CP_Elec_6.3x7.7" H 5850 3400 50  0001 C CNN
 F 3 "" H 5850 3400 50  0000 C CNN
 	1    5850 3400
@@
 F 0 "LS1" H 5850 4275 50  0000 R CNN
 F 1 "Speaker" H 5850 4200 50  0000 R CNN
-F 2 "Oddities:NetTie-I_SMD" H 5800 3850 50  0001 C CNN
+F 2 "SurfaceConnector:Surface Connector" H 5800 3850 50  0001 C CNN
 F 3 "" H 5790 4000 50  0000 C CNN
 	1    5800 4050
@@
 L Device:LED D1
 U 1 1 5BA69078
-P 6100 2950
-F 0 "D1" H 6100 3050 50  0000 C CNN
-F 1 "LED" H 6100 2850 50  0000 C CNN
-F 2 "Capacitors_SMD:C_0805" H 6100 2950 50  0001 C CNN
-F 3 "" H 6100 2950 50  0000 C CNN
-	1    6100 2950
-	-1   0    0    1
+P 3875 3000
+F 0 "D1" H 3875 3100 50  0000 C CNN
+F 1 "LED" H 3875 2900 50  0000 C CNN
+F 2 "LED_THT:LED_D5.0mm_Clear" H 3875 3000 50  0001 C CNN
+F 3 "" H 3875 3000 50  0000 C CNN
+	1    3875 3000
+	0    -1   -1   0
 $EndComp
 $Comp
 L Device:R R1
 U 1 1 5BA690F1
-P 5550 2950
-F 0 "R1" V 5630 2950 50  0000 C CNN
-F 1 "10k" V 5550 2950 50  0000 C CNN
-F 2 "Resistors_SMD:R_0805_HandSoldering" V 5480 2950 50  0001 C CNN
-F 3 "" H 5550 2950 50  0000 C CNN
-	1    5550 2950
-	0    1    1    0
+P 3875 2700
+F 0 "R1" V 3955 2700 50  0000 C CNN
+F 1 "10k" V 3875 2700 50  0000 C CNN
+F 2 "Resistor_SMD:R_0603_1608Metric" V 3805 2700 50  0001 C CNN
+F 3 "" H 3875 2700 50  0000 C CNN
+	1    3875 2700
+	1    0    0    -1
 $EndComp
 $Comp
 L power:GND #PWR02
 U 1 1 5BA6927E
-P 6700 3100
-F 0 "#PWR02" H 6700 2850 50  0001 C CNN
-F 1 "GND" H 6700 2950 50  0000 C CNN
-F 2 "" H 6700 3100 50  0000 C CNN
-F 3 "" H 6700 3100 50  0000 C CNN
-	1    6700 3100
+P 3875 3150
+F 0 "#PWR02" H 3875 2900 50  0001 C CNN
+F 1 "GND" H 3875 3000 50  0000 C CNN
+F 2 "" H 3875 3150 50  0000 C CNN
+F 3 "" H 3875 3150 50  0000 C CNN
+	1    3875 3150
 	1    0    0    -1
 $EndComp
@@
 $EndComp
 $Comp
-L The-Ear-Tool-rescue:CONN_01X02 P3
+L The-Ear-Tool-rescue:CONN_01X02-The-Ear-Tool-rescue P3
 U 1 1 5BA6951F
 P 8600 3850
 F 0 "P3" H 8600 4000 50  0000 C CNN
 F 1 "9V Battery Clip" H 8600 3700 50  0000 C CNN
-F 2 "Oddities:NetTie-I_SMD" H 8600 3850 50  0001 C CNN
+F 2 "SurfaceConnector:Surface Connector" H 8600 3850 50  0001 C CNN
 F 3 "" H 8600 3850 50  0000 C CNN
 	1    8600 3850
@@
 $EndComp
 $Comp
-L Switch1:SW_DPDT_x2 SW1
+L The-Ear-Tool-rescue:SW_DPDT_x2-Switch1 SW1
 U 1 1 5BA6D851
-P 4550 2850
-F 0 "SW1" H 4550 3020 50  0000 C CNN
-F 1 "Power Switch" H 4550 2650 50  0000 C CNN
-F 2 "myFootprints:SW_SPDT_3P_11.1mm_5.5mm" H 4550 2850 50  0001 C CNN
-F 3 "" H 4550 2850 50  0001 C CNN
-	1    4550 2850
-	1    0    0    -1
-$EndComp
-$Comp
-L Switch1:SW_DPDT_x2 SW2
+P 3475 2400
+F 0 "SW1" H 3475 2570 50  0000 C CNN
+F 1 "Power Switch" H 3475 2200 50  0000 C CNN
+F 2 "Switch:SPDT_generic_toggle" H 3475 2400 50  0001 C CNN
+F 3 "" H 3475 2400 50  0001 C CNN
+	1    3475 2400
+	1    0    0    -1
+$EndComp
+$Comp
+L The-Ear-Tool-rescue:SW_DPDT_x2-Switch1 SW2
 U 1 1 5BA6D982
 P 4550 4050
 F 0 "SW2" H 4550 4220 50  0000 C CNN
 F 1 "Full Scope Switch" H 4550 3850 50  0000 C CNN
-F 2 "myFootprints:SW_SPDT_3P_11.1mm_5.5mm" H 4550 4050 50  0001 C CNN
+F 2 "Switch:SPDT_generic_toggle" H 4550 4050 50  0001 C CNN
 F 3 "" H 4550 4050 50  0001 C CNN
 	1    4550 4050
@@
 Text GLabel 4900 3500 0    60   Input ~ 0
 SENSE
-NoConn ~ 4750 2750
+NoConn ~ 3675 2300
 NoConn ~ 4750 3950
 $Comp
-L The-Ear-Tool-rescue:CONN_01X02 P2
+L The-Ear-Tool-rescue:CONN_01X02-The-Ear-Tool-rescue P2
 U 1 1 5BAC28C2
 P 8600 2900
 F 0 "P2" H 8600 3050 50  0000 C CNN
 F 1 "Sensor Connector" H 8600 2750 50  0000 C CNN
-F 2 "Oddities:NetTie-I_SMD" H 8600 2900 50  0001 C CNN
+F 2 "TerminalBlock_RND:TerminalBlock_RND_205-00232_Pitch5.08mm" H 8600 2900 50  0001 C CNN
 F 3 "" H 8600 2900 50  0000 C CNN
 	1    8600 2900
@@
 $EndComp
 $Comp
-L The-Ear-Tool-rescue:AUDIO-JACK-3F07-TRS P1
+L The-Ear-Tool-rescue:AUDIO-JACK-3F07-TRS-The-Ear-Tool-rescue P1
 U 1 1 5BAC44CA
 P 6800 3950
 F 0 "P1" H 6700 3600 60  0000 L CNN
 F 1 "AUDIO-JACK-3F07-TRS" H 6150 4300 60  0000 L CNN
-F 2 "Connectors:AUDIO-JACK-3F07-TRS" H 6650 3800 60  0001 C CNN
+F 2 "myFootprints:AUDIO-JACK-3F07-TRS" H 6650 3800 60  0001 C CNN
 F 3 "" H 6650 3800 60  0000 C CNN
 	1    6800 3950
@@
 $EndComp
 $Comp
-L The-Ear-Tool-rescue:POT RV1
+L The-Ear-Tool-rescue:POT-The-Ear-Tool-rescue RV1
 U 1 1 5BAC4D81
 P 8050 2850
 F 0 "RV1" V 7950 2850 50  0000 C CNN
 F 1 "10k" V 8050 2850 50  0000 C CNN
-F 2 "myFootprints:POT_RV09_HORIZONTAL_WHO9" H 8050 2850 50  0001 C CNN
+F 2 "Potentiometer_THT:Potentiometer_Bourns_PTV09A-1_Single_Vertical" H 8050 2850 50  0001 C CNN
 F 3 "" H 8050 2850 50  0000 C CNN
 	1    8050 2850
-	0    -1   -1   0
+	0    1    -1   0
 $EndComp
 $Comp
 L power:+9V #PWR07
 U 1 1 5BAD0A95
-P 4200 2700
-F 0 "#PWR07" H 4200 2550 50  0001 C CNN
-F 1 "+9V" H 4200 2840 50  0000 C CNN
-F 2 "" H 4200 2700 50  0000 C CNN
-F 3 "" H 4200 2700 50  0000 C CNN
-	1    4200 2700
+P 3125 2250
+F 0 "#PWR07" H 3125 2100 50  0001 C CNN
+F 1 "+9V" H 3125 2390 50  0000 C CNN
+F 2 "" H 3125 2250 50  0000 C CNN
+F 3 "" H 3125 2250 50  0000 C CNN
+	1    3125 2250
 	1    0    0    -1
 $EndComp
@@
 F 0 "R2" V 6330 4150 50  0000 C CNN
 F 1 "100" V 6250 4150 50  0000 C CNN
-F 2 "Resistors_SMD:R_0805_HandSoldering" V 6180 4150 50  0001 C CNN
+F 2 "Resistor_SMD:R_0603_1608Metric" V 6180 4150 50  0001 C CNN
 F 3 "" H 6250 4150 50  0000 C CNN
 	1    6250 4150
@@
 	5500 3400 5700 3400
 Wire Wire Line
-	4750 2950 5100 2950
-Wire Wire Line
 	6000 3400 6300 3400
 Wire Wire Line
-	4200 2850 4200 2700
-Connection ~ 5100 2950
-Wire Wire Line
-	5700 2950 5950 2950
-Wire Wire Line
-	6250 2950 6700 2950
-Wire Wire Line
-	6700 2950 6700 3100
+	3125 2400 3125 2250
 Wire Wire Line
 	8400 3800 8200 3800
@@
 	6100 4050 6100 4150
 Wire Wire Line
-	4200 2850 4350 2850
+	3125 2400 3275 2400
 Wire Wire Line
 	4200 3300 4200 4050
@@
 	6000 3950 6100 3950
 Wire Wire Line
-	5100 3100 5100 2950
-Wire Wire Line
 	6100 3850 6400 3850
 Wire Wire Line
@@
 	8050 2650 8050 2700
 $Comp
-L Switch1:SW_DPDT_x2 SW3
+L The-Ear-Tool-rescue:SW_DPDT_x2-Switch1 SW3
 U 1 1 5C2EC483
 P 4600 5050
 F 0 "SW3" H 4550 5200 50  0000 C CNN
 F 1 "Gain Switch" H 4600 4850 50  0000 C CNN
-F 2 "myFootprints:SW_SPDT_3P_11.1mm_5.5mm" H 4600 5050 50  0001 C CNN
+F 2 "Switch:SPDT_generic_toggle" H 4600 5050 50  0001 C CNN
 F 3 "" H 4600 5050 50  0001 C CNN
 	1    4600 5050
@@
 F 0 "C1" H 4450 4850 50  0000 L CNN
 F 1 "4.7uF" H 4300 4600 50  0000 L CNN
-F 2 "Capacitors_SMD:C_0805_HandSoldering" H 4588 4550 50  0001 C CNN
+F 2 "Capacitor_SMD:C_0603_1608Metric" H 4588 4550 50  0001 C CNN
 F 3 "" H 4550 4700 50  0001 C CNN
 	1    4550 4700
@@
 NoConn ~ 4800 4950
 Wire Wire Line
-	5100 2950 5400 2950
-Wire Wire Line
 	6300 3750 6300 4050
 Wire Wire Line
@@
 Wire Wire Line
 	5100 4150 5100 4200
+$Comp
+L Device:C_Small C3
+U 1 1 61B8A6BF
+P 4850 2975
+F 0 "C3" H 4758 2929 50  0000 R CNN
+F 1 "0u1" H 4758 3020 50  0000 R CNN
+F 2 "Capacitor_SMD:C_0603_1608Metric" H 4850 2975 50  0001 C CNN
+F 3 "~" H 4850 2975 50  0001 C CNN
+	1    4850 2975
+	1    0    0    1
+$EndComp
+Wire Wire Line
+	3675 2500 3875 2500
+$Comp
+L power:GND #PWR0101
+U 1 1 61B9075C
+P 4850 3075
+F 0 "#PWR0101" H 4850 2825 50  0001 C CNN
+F 1 "GND" H 4850 2925 50  0000 C CNN
+F 2 "" H 4850 3075 50  0000 C CNN
+F 3 "" H 4850 3075 50  0000 C CNN
+	1    4850 3075
+	1    0    0    -1
+$EndComp
+Wire Wire Line
+	4850 2875 5100 2875
+Connection ~ 5100 2875
+Wire Wire Line
+	5100 2875 5100 2500
+Wire Wire Line
+	5100 2875 5100 3100
+Wire Wire Line
+	3875 2550 3875 2500
+Connection ~ 3875 2500
+Wire Wire Line
+	3875 2500 5100 2500
 $EndSCHEMATC
